Commit message: new

File: .history/models/r2d2_20240412094135.urdf (robot description, URDF)
Before this commit: robot atirobot, 5 links, 4 joints
Joints:
- joint base_footprint_joint: origin xyz=0.0 0.0 0.73 rpy=0 0 ${pi} -> xyz=0.0 0.0 0.0 rpy=0 0 0
- joint lidar_left_joint: origin xyz=-0.3975 0.265 -0.44 rpy=0 0 ${pi/2} -> xyz=-0.31 0.2 -0.44 rpy=0 0 ${-pi/2}
- joint merged_lidar_joint: child merged_lidar_frame -> laser_frame

File: .history/models/r2d2_20240412094239.urdf (robot description, URDF)
Before this commit: robot atirobot, 5 links, 4 joints
Links:
- removed link merged_lidar_frame
- added link laser_frame, mass 0.114; collision cylinder length=0.03 radius=0.0508; visual cylinder length=0.03 radius=0.0508
Joints:
- joint base_footprint_joint: origin xyz=0.0 0.0 0.73 rpy=0 0 ${pi} -> xyz=0.0 0.0 0.0 rpy=0 0 0
- joint lidar_left_joint: origin xyz=-0.3975 0.265 -0.44 rpy=0 0 ${pi/2} -> xyz=-0.31 0.2 -0.44 rpy=0 0 ${-pi/2}
- joint merged_lidar_joint: child merged_lidar_frame -> laser_frame; origin xyz=0.0 0.0 0.35 rpy=0 0 0 -> xyz=0.0 0.0 -0.44 rpy=0 0 0
