Commit message: commit

File: models/penteknemelbaszotturdf.urdf (robot description, URDF)
Before this commit: robot vikirobot, 6 links, 5 joints
Links:
- removed link caster_wheel
- link base_link: mass 100.0 -> 205.727203925287; geometry collision mesh filename=package://r2d2/meshes/robotbase.stl; visual mesh filename=package://r2d2/meshes/robotbase.stl
- link laser_frame: geometry collision cylinder length=0.03 radius=0.0508; visual cylinder length=0.03 radius=0.0508
- link lidarleft: geometry collision cylinder length=0.03 radius=0.0508; visual cylinder length=0.03 radius=0.0508
- link lidarright: geometry collision cylinder length=0.03 radius=0.0508; visual cylinder length=0.03 radius=0.0508
Joints:
- removed joint base_caster_wheel_joint
- joint base_footprint_joint: origin xyz=-0.15 0 ${(base_height/2)+wheel_radius} rpy=0 0 0 -> xyz=0.0 0.0 0.0 rpy=0 0 0
- joint lidar_left_joint: origin xyz=-0.31 0.2 -${(base_height/2)-0.07} rpy=0 0 ${-pi/2} -> xyz=-0.31 0.2 -0.44 rpy=0 0 ${-pi/2}
- joint lidar_right_joint: origin xyz=0.31 -0.2 -${(base_height/2)-0.07} rpy=0 0 ${-3*pi/2} -> xyz=0.31 -0.2 -0.44 rpy=0 0 ${-3*pi/2}
- joint merged_lidar_joint: origin xyz=0.0 0.0 -${(base_height/2)-0.07} rpy=0 0 0 -> xyz=0.0 0.0 -0.44 rpy=0 0 0
